Commit message: rename xarco to xacro

File: jb2a_description/urdf/jb2a.urdf.xacro (robot description, xacro)
@@ -9,6 +9,6 @@
   <xacro:property name="scale_mm2" value="${scale_mm*scale_mm}"/>
   <xacro:property name="gtoKg" value="1e-3"/>
-  <xacro:property name="angle_lim_low" value="${8/18*pi}"/>
-  <xacro:property name="angle_lim_high" value="${-8/18*pi}"/>
+  <xacro:property name="angle_lim_low" value="${-8/18*pi}"/>
+  <xacro:property name="angle_lim_high" value="${8/18*pi}"/>
   <!-- Used for every servo except the first one as it is the child in the joint relation -->
   <xacro:macro name="servo" params="name">
@@ -38,6 +38,6 @@
     </link>
   </xacro:macro>
-  <xacro:macro name="servo_joint" params="parent child offset:=37.5">
-    <joint name="${parent}_${child}_joint" type="revolute">
+  <xacro:macro name="servo_joint" params="parent arm child offset:=37.5">
+    <joint name="${parent}_${arm}_joint" type="revolute">
       <parent link="${parent}"/>
       <child link="${child}"/>
@@ -47,4 +47,13 @@
       <dynamics friction="0.7"/>
     </joint>
+    <transmission name="${parent}_${child}_trans">
+      <type> transmission_interface/SimpleTransmission</type>
+      <joint name="${parent}_${arm}_joint">
+	       <hardwareInterface>hardware_interface/EffortJointInterface</hardwareInterface>
+      </joint>
+      <actuator name="${parent}_${child}_servo">
+	       <hardwareInterface>hardware_interface/EffortJointInterface</hardwareInterface>
+      </actuator>
+    </transmission>
   </xacro:macro>
   <xacro:macro name="servo_mimic" params="parent child mimic multiplier">
@@ -255,4 +264,13 @@
       <dynamics friction="0.7"/>
     </joint>
+    <transmission name="base_servo1_trans">
+      <type> transmission_interface/SimpleTransmission</type>
+      <joint name="base_servo1_joint">
+	       <hardwareInterface>hardware_interface/EffortJointInterface</hardwareInterface>
+      </joint>
+      <actuator name="base_servo1_servo">
+	       <hardwareInterface>hardware_interface/EffortJointInterface</hardwareInterface>
+      </actuator>
+    </transmission>
     <link name="piece100">
       <inertial>
@@ -384,5 +402,5 @@
       </collision>
     </link>
-    <xacro:servo_joint parent="servo2" child="arm1-piece12"/>
+    <xacro:servo_joint parent="servo2" arm="arm1" child="arm1-piece12"/>
     <link name="arm1-piece15">
       <inertial>
@@ -468,5 +486,5 @@
       </collision>
     </link>
-    <xacro:servo_joint parent="servo4" child="arm2-piece16" offset="39.5"/>
+    <xacro:servo_joint parent="servo4" arm="arm2" child="arm2-piece16" offset="39.5"/>
     <xacro:radialBearing name="radialBearing3"/>
     <joint name="arm2-piece16_radialBearing3_joint" type="fixed">
@@ -552,5 +570,5 @@
       </collision>
     </link>
-    <xacro:servo_joint parent="servo5" child="arm3-piece17"/>
+    <xacro:servo_joint parent="servo5" arm="arm3" child="arm3-piece17"/>
     <xacro:radialBearing name="radialBearing4"/>
     <xacro:radialBearing_joint parent="radialBearing3" child="radialBearing4" mimic="servo5_arm3-piece17_joint" multiplier="-1" offset="12.5"/>
@@ -648,5 +666,5 @@
        </collision>
      </link>
-    <xacro:servo_joint parent="servo6" child="fakeHand"/>
+    <xacro:servo_joint parent="servo6" arm="hand" child="fakeHand"/>
    <!-- End hand -->
 </robot>
